Commit message: Fix URDF base frame and Nav2 acceleration limits to stop teleporting

File: install/my_robot_description/share/my_robot_description/urdf/my_robot.urdf.xacro (robot description, xacro)
@@ -29,10 +29,4 @@
     </inertial>
   </xacro:macro>
-  <link name="base_footprint"/>
-  <joint name="base_joint" type="fixed">
-    <parent link="base_footprint"/>
-    <child link="base_link"/>
-    <origin xyz="0 0 0"/>
-  </joint>
   <link name="base_link"/>
   <link name="chassis">
@@ -154,5 +148,5 @@
     </sensor>
   </gazebo>
-  <gazebo>
+ <gazebo>
     <plugin name="diff_drive" filename="libgazebo_ros_diff_drive.so">
       <left_joint>left_wheel_joint</left_joint>
@@ -166,5 +160,5 @@
       <publish_wheel_tf>true</publish_wheel_tf>
       <odometry_frame>odom</odometry_frame>
-      <robot_base_frame>base_footprint</robot_base_frame>
+      <robot_base_frame>base_link</robot_base_frame>
     </plugin>
   </gazebo>
